File: hardware/mother/main-board/standard_cell.kicad_sch (KiCad schematic)
At the start: 13 parts, among them J9 Conn_01x02_Pin, U1 DIP, U10 TL071, U2 DIP, U4 AD5263BRUZ200, U6 AD5263BRUZ200, U9 TL071

Commit message: hardware locking in
Parts:
- removed U1, U2: DIP, Package_DIP:DIP-40_W15.24mm_LongPads, symbol SeniorDesign:MTT8816DIP
- added U11, U12: CD22M3494MQZ, SeniorDesignFP:PLCC44_16P66X16P66_INR-M, symbol SeniorDesign:CD22M3494MQZ
- U8: renamed from U6; footprint Package_DIP:DIP-24_W15.24mm -> SeniorDesignFP:SOP65P640X120-24N; DKPN (none) -> AD5263BRUZ200-R7; MPN AD5263BRUZ200 -> (none)
- U9: renamed from U4; footprint Package_DIP:DIP-24_W15.24mm -> SeniorDesignFP:SOP65P640X120-24N; DKPN (none) -> AD5263BRUZ200-R7; MPN AD5263BRUZ200 -> (none)
- renumbered C19 to C1, C20 to C2, C21 to C3, C22 to C4, J9 to J5, U9 to U7
Connections:
- net C1_in: now also U12.25 (X12)
- net C1_out: now also U12.24 (X13)
- net C2_in: now also U11.2 (X14)
- net C2_out: now also U11.3 (X15)
- net C3_in: now also U11.8 (X10)
- net C3_out: now also U11.9 (X11)
- net C4_in: now also U11.6 (X8)
- net C4_out: now also U11.7 (X9)
- net D1_anode: now also U11.5 (X7)
- net D1_cathode: now also U11.4 (X6)
- net D2_anode: now also U11.24 (X13)
- net D2_cathode: now also U11.25 (X12)
- net GND: now also U11.17 (Y4), U12.32 (Y0)
- net Input_1: now also U11.32 (Y0), U12.17 (Y4)
- net Input_2: now also U11.35 (Y1), U12.15 (Y5)
- net Input_3: now also U11.37 (Y2), U12.13 (Y6)
- net J1_in: now also U11.27 (X4)
- net J1_out: now also U11.26 (X5)
- net Op1_neg: now also U12.29 (X2)
- net Op1_out: now also U12.31 (X0)
- net Op1_pos: now also U12.30 (X1)
- net Op2_neg: now also U12.27 (X4)
- net Op2_out: now also U12.28 (X3)
- net Op2_pos: now also U12.26 (X5)
- net Output: now also U11.39 (Y3), U12.10 (Y7)
- net R1_in: now also U12.5 (X7)
- net R1_out: now also U12.4 (X6)
- net R2_in: now also U12.6 (X8)
- net R2_out: now also U12.7 (X9)
- net R3_in: now also U12.3 (X15)
- net R3_out: now also U12.2 (X14)
- net R4_in: now also U12.8 (X10)
- net R4_out: now also U12.9 (X11)
- net R5_in: now also U11.31 (X0)
- net R5_out: now also U11.30 (X1)
- net R6_in: now also U11.29 (X2)
- net R6_out: now also U11.28 (X3)
- net Y5: now also U11.15 (Y5), U12.35 (Y1)
- net Y6: now also U11.13 (Y6), U12.37 (Y2)
- net Y7: now also U11.10 (Y7), U12.39 (Y3)
Other:
- title: (none) -> Standard Cell Design Schematic
- moved on the sheet: C1, C2, C3, C4, D1, D2, J5, U10, U7, U8B, U8C, U8D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
