File: hardware/daughter/main-board/MainBoard.kicad_sch (KiCad schematic)
At the start: 1 part, among them J1 Conn_01x20_Pin

Commit message: daughter board clayton edits
Changed lines of the file:
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@@
 	)
 	(sheet
-		(at 231.14 46.99)
+		(at 82.55 76.2)
 		(size 31.75 88.9)
 		(exclude_from_sim no)
@@
 		)
 		(property "Sheetname" "Microcontroller & Controls"
-			(at 231.14 46.2784 0)
+			(at 82.55 75.4884 0)
 			(effects
 				(font
@@
 		)
 		(property "Sheetfile" "stm_controls.kicad_sch"
-			(at 231.14 136.4746 0)
+			(at 82.55 165.6846 0)
 			(effects
 				(font
