File: hardware/daughter/main-board/stm_controls.kicad_sch (KiCad schematic)
At the start: 57 parts, among them J10 USB_C_Receptacle_USB2.0_14P, J11 Conn_02x05_Odd_Even, J12 Conn_01x02_Pin, J13 Conn_01x02_Pin, SW3 SW_SPST, SW4 SW_SPST, U1 CD22M3494MQZ, U11 CD22M3494MQZ, U12 CD22M3494MQZ, U14 AD5263BRUZ200, U15 AD5263BRUZ200, U17 CD22M3494MQZ, U18 CD22M3494MQZ, U20 AD5263BRUZ200, U21 AD5263BRUZ200, U23 CD22M3494MQZ, U24 CD22M3494MQZ, U26 AD5263BRUZ200, U27 AD5263BRUZ200, U29 CD22M3494MQZ, U30 CD22M3494MQZ, U34 74HC164, U35 FT232RL, U36 74HC164, U37 STM32F091RCTx, U38 74HC164, U8 AD5263BRUZ200, U9 AD5263BRUZ200

Commit message: daughter board clayton edits
Parts:
- removed C20, C23, C24, C25: 100nF, Capacitor_SMD:C_0603_1608Metric_Pad1.08x0.95mm_HandSolder, symbol Device:C
- removed C22: 10µF, Capacitor_SMD:C_0603_1608Metric_Pad1.08x0.95mm_HandSolder, symbol Device:C
- removed C28: 10nF, Capacitor_SMD:C_0603_1608Metric_Pad1.08x0.95mm_HandSolder, symbol Device:C
- removed C29: 1µF, Capacitor_SMD:C_0603_1608Metric_Pad1.08x0.95mm_HandSolder, symbol Device:C
- removed D10: GREENLED, Diode_SMD:D_0805_2012Metric_Pad1.15x1.40mm_HandSolder, symbol Device:LED
- removed D11: BAT60JFILM, Diode_SMD:D_SOD-323_HandSoldering, symbol Device:D_Schottky
- removed D9: REDLED, Diode_SMD:D_0805_2012Metric_Pad1.15x1.40mm_HandSolder, symbol Device:LED
- removed F4: 500mA, Fuse:Fuse_0603_1608Metric_Pad1.05x0.95mm_HandSolder, symbol Device:Fuse
- removed J10: USB_C_Receptacle_USB2.0_14P, Connector_USB:USB_C_Receptacle_G-Switch_GT-USB-7010ASV, symbol Connector:USB_C_Receptacle_USB2.0_14P
- removed J12, J13: Conn_01x02_Pin, Connector_PinSocket_2.54mm:PinSocket_1x02_P2.54mm_Vertical, symbol Connector:Conn_01x02_Pin
- removed R1, R4: 150Ω, Resistor_SMD:R_0603_1608Metric_Pad0.98x0.95mm_HandSolder, symbol Device:R_US
- removed R2, R3: 10k, Resistor_SMD:R_0603_1608Metric_Pad0.98x0.95mm_HandSolder, symbol Device:R_US
- removed R5, R8: 10kΩ, Resistor_SMD:R_0603_1608Metric_Pad0.98x0.95mm_HandSolder, symbol Device:R_US
- removed SW4: SW_SPST, Button_Switch_SMD:SW_SPST_SKQG_WithoutStem, symbol Switch:SW_SPST
- removed U12, U18, U23, U29, U30: CD22M3494MQZ, SeniorDesignFP:PLCC44_16P66X16P66_INR-M, symbol SeniorDesign:CD22M3494MQZ
- removed U34, U36, U38: 74HC164, Package_SO:SOIC-14_3.9x8.7mm_P1.27mm, symbol 74xx:74HC164
- removed U35: FT232RL, Package_SO:SSOP-28_5.3x10.2mm_P0.65mm, symbol Interface_USB:FT232RL
- removed U37: STM32F091RCTx, Package_QFP:LQFP-64_10x10mm_P0.5mm, symbol MCU_ST_STM32F0:STM32F091RCTx
- added C5: 100nF, Capacitor_SMD:C_0603_1608Metric_Pad1.08x0.95mm_HandSolder, symbol Device:C
- added U10, U12, U5, U6, U7: ADG1414BRUZ, symbol SeniorDesign:ADG1414BRU_1
- added U13: 74HC138, symbol 74xx:74HC138
- added U3: STM32C092CBT6, LQFP48_STM, symbol SeniorDesign:STM32C092CBT6
- C21: value 10µF -> 4.7µF
Connections:
- net +3.3V: now also U13.16 (VCC); no longer C21.1, C26.1, C27.1
- net GND: now also C5.2, U13.4 (~{E0}), U13.5 (~{E1}), U13.8 (GND), U3.7 (VSS/VSSA)
- net LED_STM_1: now also U3.40 (PD2)
- net LED_STM_2: now also U3.39 (PD1)
- net LED_STM_3: now also U3.38 (PD0)
- net MT_AX0: now also U3.24 (PB12)
- net MT_AX1: now also U3.25 (PB13)
- net MT_AX2: now also U3.26 (PB14)
- net MT_AX3: now also U3.27 (PB15)
- net MT_AY0: now also U3.21 (PB2)
- net MT_AY1: now also U3.22 (PB10)
- net MT_AY2: now also U3.23 (PB11)
- net MT_DAT: now also U3.44 (PB5)
- net MT_RST: now also U3.43 (PB4)
- net MT_STB: now also U3.42 (PB3)
- net SPI1_MOSI: now also U3.18 (PA7)
- net SPI1_SCK: now also U3.16 (PA5)
- net SWCLK: now also U3.36 (PA14-BOOT0)
- net SWDIO: now also U3.35 (PA13)
- net +3.3VA: no longer names the net of FB1.1
- net +3.3VA: now also C21.1, C26.1, C27.1, U3.5 (VREF+), U3.6 (VDD/VDDA)
- net NRST renamed RST
- net RST: now also C5.1, U3.10 (PF2-NRST)
- new net CM_A0: U13.1 (A0), U3.28 (PA8)
- new net CM_A1: U13.2 (A1), U3.29 (PA9)
- new net CM_A2: U13.3 (A2), U3.32 (PA10)
- new net CM_DPOT_CS0: U13.10 (~{Y5})
- new net CM_DPOT_CS1: U13.9 (~{Y6})
- new net CM_DPOT_CS2: U13.7 (~{Y7})
- new net CM_EN: U13.6 (E2), U3.33 (PA11[PA9])
- new net CM_SPST_CS0: U13.15 (~{Y0}), U5.24 (~SYNC)
- new net CM_SPST_CS1: U13.14 (~{Y1}), U6.24 (~SYNC)
- new net CM_SPST_CS2: U10.24 (~SYNC), U13.13 (~{Y2})
- new net CM_SPST_CS3: U12.24 (~SYNC), U13.12 (~{Y3})
- new net CM_SPST_CS4: U13.11 (~{Y4}), U7.24 (~SYNC)
- new net DATA_READY: U3.31 (PC7)
- new net GPIO: U3.1 (PC13)
- new net MT_CS0: U3.11 (PA0)
- new net MT_CS1: U3.12 (PA1)
- new net MT_CS2: U3.13 (PA2)
- new net MT_CS3: U3.14 (PA3)
- new net SPI1_MISO: U3.17 (PA6)
- new net SPI1_NSS: U3.15 (PA4)
- new net SPI2_MISO: U3.45 (PB6)
- new net SPI2_MOSI: U10.3 (DIN), U12.3 (DIN), U3.46 (PB7), U5.3 (DIN), U6.3 (DIN), U7.3 (DIN)
- new net SPI2_NSS: U3.48 (PB9)
- new net SPI2_SCK: U10.1 (SCLK), U12.1 (SCLK), U3.47 (PB8), U5.1 (SCLK), U7.1 (SCLK)
- new net STS: U3.30 (PC6)
- no-connect marks 59 -> 33
Other:
- moved on the sheet: C21, C26, C27, C30, D12, D13, D14, FB1, J11, R10, R6, R7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
